File: sdcard_sensor/sdcard_sensor.kicad_pcb (KiCad board)
At the start: 2 copper layers, 37.9 x 26.1 mm, 1 part, among them X1 microSD_Card

Commit message: Format changed
Other:
- board size 37.9 x 26.1 mm -> 35.9 x 11 mm
Changed lines of the file:
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@@
 (kicad_pcb (version 20171130) (host pcbnew 5.1.9)
   (general
-    (thickness 1.6)
-    (drawings 20)
+    (thickness 0.8)
+    (drawings 16)
     (tracks 0)
     (zones 0)
@@
       (effects (font (size 1 1) (thickness 0.15)))
     )
+    (fp_line (start 7.5 4.9) (end -7.5 4.9) (layer F.SilkS) (width 0.05))
+    (fp_line (start 7.5 -6.1) (end 7.5 4.9) (layer F.SilkS) (width 0.05))
+    (fp_line (start -2.7 -4.8) (end -7.5 -4.8) (layer F.SilkS) (width 0.05))
+    (fp_line (start -7.5 -4.8) (end -7.5 4.9) (layer F.SilkS) (width 0.05))
+    (fp_line (start 1.1 -5.3) (end -0.1 -5.3) (layer F.SilkS) (width 0.05))
+    (fp_line (start -0.1 -5.9) (end -1.6 -5.9) (layer F.SilkS) (width 0.05))
+    (fp_line (start -2.7 -4.8) (end -1.6 -5.9) (layer F.SilkS) (width 0.05))
+    (fp_line (start 1.1 -5.3) (end 1.9 -6.1) (layer F.SilkS) (width 0.05))
+    (fp_line (start 1.9 -6.1) (end 7.5 -6.1) (layer F.SilkS) (width 0.05))
     (fp_line (start -0.1 -5.9) (end -0.1 -5.3) (layer F.SilkS) (width 0.05))
-    (fp_line (start 1.9 -6.1) (end 7.5 -6.1) (layer F.SilkS) (width 0.05))
-    (fp_line (start 1.1 -5.3) (end 1.9 -6.1) (layer F.SilkS) (width 0.05))
-    (fp_line (start -2.7 -4.8) (end -1.6 -5.9) (layer F.SilkS) (width 0.05))
-    (fp_line (start -0.1 -5.9) (end -1.6 -5.9) (layer F.SilkS) (width 0.05))
-    (fp_line (start 1.1 -5.3) (end -0.1 -5.3) (layer F.SilkS) (width 0.05))
-    (fp_line (start -7.5 -4.8) (end -7.5 4.9) (layer F.SilkS) (width 0.05))
-    (fp_line (start -2.7 -4.8) (end -7.5 -4.8) (layer F.SilkS) (width 0.05))
-    (fp_line (start 7.5 -6.1) (end 7.5 4.9) (layer F.SilkS) (width 0.05))
-    (fp_line (start 7.5 4.9) (end -7.5 4.9) (layer F.SilkS) (width 0.05))
     (pad 8 smd rect (at -4.95 3.9 270) (size 0.8 2.9) (layers B.Cu B.Paste B.Mask)
       (net 1 "Net-(X1-Pad8)"))
@@
       (net 8 "Net-(X1-Pad1)"))
   )
-  (gr_line (start 137.3 73.9) (end 156 73.9) (layer Edge.Cuts) (width 0.05))
-  (gr_line (start 137.3 79.9) (end 137.3 73.9) (layer Edge.Cuts) (width 0.05))
-  (gr_line (start 136 81.2) (end 137.3 79.9) (layer Edge.Cuts) (width 0.05))
-  (gr_line (start 156 100) (end 156 73.9) (layer Edge.Cuts) (width 0.05))
-  (gr_line (start 137.3 100) (end 156 100) (layer Edge.Cuts) (width 0.05))
-  (gr_line (start 137.3 93.5) (end 137.3 100) (layer Edge.Cuts) (width 0.05))
-  (gr_line (start 136 92.2) (end 137.3 93.5) (layer Edge.Cuts) (width 0.05))
-  (gr_line (start 133.1 92.2) (end 136 92.2) (layer Edge.Cuts) (width 0.05))
-  (gr_line (start 133.1 81.2) (end 136 81.2) (layer Edge.Cuts) (width 0.05))
+  (gr_arc (start 153 91.2) (end 153 92.2) (angle -90) (layer Edge.Cuts) (width 0.05))
+  (gr_arc (start 153 82.2) (end 154 82.2) (angle -90) (layer Edge.Cuts) (width 0.05))
+  (gr_line (start 153 92.2) (end 133.1 92.2) (layer Edge.Cuts) (width 0.05))
+  (gr_line (start 154 82.2) (end 154 91.2) (layer Edge.Cuts) (width 0.05))
+  (gr_line (start 133.1 81.2) (end 153 81.2) (layer Edge.Cuts) (width 0.05))
   (gr_arc (start 118.4 91.9) (end 118.1 91.9) (angle -90) (layer Edge.Cuts) (width 0.05))
   (gr_arc (start 118.4 82.8) (end 118.4 82.5) (angle -90) (layer Edge.Cuts) (width 0.05))

Commit message: Template done
Parts:
- added C1: 100nF, Capacitor_SMD:C_0402_1005Metric, F.Cu at (138.7, 86.7)
- added J1: Conn_02x04_Counter_Clockwise, Connector_PinSocket_2.00mm:PinSocket_2x04_P2.00mm_Vertical, F.Cu at (136.8, 83.7)
Connections:
- X1 pad 1: Net-(X1-Pad1) -> DAT2
- X1 pad 2: Net-(X1-Pad2) -> DAT3
- X1 pad 3: Net-(X1-Pad3) -> CMD
- X1 pad 4: Net-(X1-Pad4) -> +3V3
- X1 pad 5: Net-(X1-Pad5) -> CLK
- X1 pad 6: Net-(X1-Pad6) -> GND
- X1 pad 7: Net-(X1-Pad7) -> DAT0
- X1 pad 8: Net-(X1-Pad8) -> DAT1
Routing:
- net CLK: track 0.00 -> 23.1 mm, vias 0 -> 1
- net DAT2: track 0.00 -> 18.1 mm
- net DAT0: track 0.00 -> 17.1 mm
- net CMD: track 0.00 -> 17.0 mm, vias 0 -> 1
- net +3V3: track 0.00 -> 15.8 mm, vias 0 -> 1
- net GND: track 0.00 -> 14.8 mm
- net DAT1: track 0.00 -> 14.8 mm
- net DAT3: track 0.00 -> 14.5 mm
- added copper zone on B.Cu, net +3V3
- added copper zone on F.Cu, net GND
Other:
- rule pad_to_mask_clearance: 0 -> 0.051
- rule trace_min: 0.2 -> 0.127
- rule via_min_size: 0.4 -> 0.6
- board text added: "DAT2 CD/DAT3 CMD 3V3 CLK GND DAT0 DAT1"
- board text added: "J1 Pinout Model D3/SDA - D2/SCL 3V3 - CMD GND - CLK D1 - D0"
- board text added: "MicroSD Module Sensor"
- board text added: "MicroSD Sensor Module"
